File: IC60/IC60.kicad_pcb (KiCad board)
At the start: 2 copper layers, 285 x 95 mm, 161 parts, among them J1 USB_CONN, P1 DEBUG, P2 CONN_2, P3 FLASH_HDR, U1 MK20LF

Commit message: Remove unneeded footprints and tweak the netlist a bit to fix for the correct new usb module.
Parts:
- Ss15: footprint lib.pretty:MXALPS -> lib.pretty:MXALPS_HIDDEN
Changed lines of the file:
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@@
     (links 261)
     (no_connects 9)
-    (area 56.622387 63.5176 353.973513 160.3906)
+    (area 62.243969 63.870469 347.331031 158.958281)
     (thickness 1.6002)
     (drawings 19)
@@
     )
   )
-  (module lib.pretty:MXALPS (layer Front)
-    (at 328.613 73.82)
-    (descr MXALPS)
-    (tags MXALPS)
-    (fp_text reference Ss15 (at 0 -2.54) (layer B.SilkS) hide
-      (effects (font (size 1 1) (thickness 0.2)) (justify mirror))
-    )
-    (fp_text value SW (at -3.5 9) (layer B.SilkS) hide
-      (effects (font (thickness 0.3048)) (justify mirror))
-    )
-    (fp_line (start -7.75 6.4) (end -7.75 -6.4) (layer Dwgs.User) (width 0.3))
-    (fp_line (start -7.75 6.4) (end 7.75 6.4) (layer Dwgs.User) (width 0.3))
-    (fp_line (start 7.75 6.4) (end 7.75 -6.4) (layer Dwgs.User) (width 0.3))
-    (fp_line (start 7.75 -6.4) (end -7.75 -6.4) (layer Dwgs.User) (width 0.3))
-    (fp_line (start -7.62 -7.62) (end 7.62 -7.62) (layer Dwgs.User) (width 0.3))
-    (fp_line (start 7.62 -7.62) (end 7.62 7.62) (layer Dwgs.User) (width 0.3))
-    (fp_line (start 7.62 7.62) (end -7.62 7.62) (layer Dwgs.User) (width 0.3))
-    (fp_line (start -7.62 7.62) (end -7.62 -7.62) (layer Dwgs.User) (width 0.3))
-    (pad "" np_thru_hole circle (at 0 0) (size 3.98781 3.98781) (drill 3.9878) (layers *.Cu *.Mask F.SilkS)
-      (clearance 0.1524))
-    (pad "" np_thru_hole circle (at -5.08 0) (size 1.70181 1.70181) (drill 1.7018) (layers *.Cu *.Mask F.SilkS)
-      (clearance 0.1524))
-    (pad "" np_thru_hole circle (at 5.08 0) (size 1.70181 1.70181) (drill 1.7018) (layers *.Cu *.Mask F.SilkS)
-      (clearance 0.1524))
-    (pad 1 thru_hole oval (at -3.405 -3.27 330.95) (size 2.5 4.17) (drill oval 1.5 3.17) (layers *.Cu *.Mask F.SilkS)
-      (net 7 /matrix/Col6))
-    (pad 2 thru_hole oval (at 2.52 -4.79 356.1) (size 2.5 3.08) (drill oval 1.5 2.08) (layers *.Cu *.Mask F.SilkS)
-      (net 44 "Net-(D15-Pad1)"))
-  )
   (module lib.pretty:SOT123-DIODE (layer Back)
     (at 74.549 73.8188)
@@
       (net 92 "Net-(D63-Pad1)"))
   )
+  (module lib.pretty:MXALPS_HIDDEN (layer Front)
+    (at 328.613 73.82)
+    (descr MXALPS)
+    (tags MXALPS)
+    (fp_text reference Ss15 (at 0 -2.54) (layer B.SilkS) hide
+      (effects (font (size 1 1) (thickness 0.2)) (justify mirror))
+    )
+    (fp_text value SW (at -3.5 9) (layer B.SilkS) hide
+      (effects (font (thickness 0.3048)) (justify mirror))
+    )
+    (fp_line (start -7.75 6.4) (end -7.75 -6.4) (layer Dwgs.User) (width 0.3))
+    (fp_line (start -7.75 6.4) (end 7.75 6.4) (layer Dwgs.User) (width 0.3))
+    (fp_line (start 7.75 6.4) (end 7.75 -6.4) (layer Dwgs.User) (width 0.3))
+    (fp_line (start 7.75 -6.4) (end -7.75 -6.4) (layer Dwgs.User) (width 0.3))
+    (fp_line (start -7.62 -7.62) (end 7.62 -7.62) (layer Dwgs.User) (width 0.3))
+    (fp_line (start 7.62 -7.62) (end 7.62 7.62) (layer Dwgs.User) (width 0.3))
+    (fp_line (start 7.62 7.62) (end -7.62 7.62) (layer Dwgs.User) (width 0.3))
+    (fp_line (start -7.62 7.62) (end -7.62 -7.62) (layer Dwgs.User) (width 0.3))
+    (pad "" np_thru_hole circle (at 0 0) (size 3.98781 3.98781) (drill 3.9878) (layers *.Cu *.Mask F.SilkS)
+      (clearance 0.1524))
+    (pad "" np_thru_hole circle (at -5.08 0) (size 1.70181 1.70181) (drill 1.7018) (layers *.Cu *.Mask F.SilkS)
+      (clearance 0.1524))
+    (pad "" np_thru_hole circle (at 5.08 0) (size 1.70181 1.70181) (drill 1.7018) (layers *.Cu *.Mask F.SilkS)
+      (clearance 0.1524))
+    (pad 1 thru_hole oval (at -3.405 -3.27 330.95) (size 2.5 4.17) (drill oval 1.5 3.17) (layers *.Cu *.Mask F.SilkS)
+      (net 7 /matrix/Col6))
+    (pad 2 thru_hole oval (at 2.52 -4.79 356.1) (size 2.5 3.08) (drill oval 1.5 2.08) (layers *.Cu *.Mask F.SilkS)
+      (net 44 "Net-(D15-Pad1)"))
+  )
   (gr_line (start 75.51 64.92875) (end 64.3255 64.92875) (angle 90) (layer Edge.Cuts) (width 0.09906))

Commit message: IC60 1.1a, now with moar LEDs.
Parts:
- removed D64: LED, lib.pretty:LED-0603
- removed the P1 at (90.6, 113.2)
- added C7: 0.1uF, lib.pretty:SMD-1005, B.Cu at (158.7, 141.9)
- added C8: 0.1uF, lib.pretty:SMD-1005, B.Cu at (163.4, 146.0)
- added LED1: LED, lib.pretty:INSW_LEDS, F.Cu at (71.4, 68.7)
- added LED10: LED, lib.pretty:INSW_LEDS, F.Cu at (242.9, 68.7)
- added LED11: LED, lib.pretty:INSW_LEDS, F.Cu at (261.9, 68.7)
- added LED114: LED, lib.pretty:INSW_LEDS_HIDDEN, F.Cu at (328.6, 68.7)
- added LED12: LED, lib.pretty:INSW_LEDS, F.Cu at (281.0, 68.7)
- added LED13: LED, lib.pretty:INSW_LEDS, F.Cu at (300.0, 68.7)
- added LED14: LED, lib.pretty:INSW_LEDS, F.Cu at (319.1, 68.7)
- added LED15: LED, lib.pretty:INSW_LEDS, F.Cu at (338.1, 68.7)
- added LED154: LED, lib.pretty:INSW_LEDS_HIDDEN, F.Cu at (321.5, 125.9)
- added LED156: LED, lib.pretty:INSW_LEDS_HIDDEN, F.Cu at (76.2, 144.9)
- added LED157: LED, lib.pretty:INSW_LEDS_HIDDEN, F.Cu at (100.0, 144.9)
- added LED158: LED, lib.pretty:INSW_LEDS_HIDDEN, F.Cu at (123.8, 144.9)
- added LED159: LED, lib.pretty:INSW_LEDS_HIDDEN, F.Cu at (195.3, 144.9)
- added LED16: LED, lib.pretty:INSW_LEDS, F.Cu at (76.2, 87.8)
- added LED160: LED, lib.pretty:INSW_LEDS_HIDDEN, F.Cu at (266.7, 144.9)
- added LED161: LED, lib.pretty:INSW_LEDS_HIDDEN, F.Cu at (290.5, 144.9)
- added LED162: LED, lib.pretty:INSW_LEDS_HIDDEN, F.Cu at (311.9, 144.9)
- added LED163: LED, lib.pretty:INSW_LEDS_HIDDEN, F.Cu at (335.8, 144.9)
- added LED17: LED, lib.pretty:INSW_LEDS, F.Cu at (100.0, 87.8)
- added LED18: LED, lib.pretty:INSW_LEDS, F.Cu at (119.1, 87.8)
- added LED19: LED, lib.pretty:INSW_LEDS, F.Cu at (138.1, 87.8)
- added LED2: LED, lib.pretty:INSW_LEDS, F.Cu at (90.5, 68.7)
- added LED20: LED, lib.pretty:INSW_LEDS, F.Cu at (157.2, 87.8)
- added LED21: LED, lib.pretty:INSW_LEDS, F.Cu at (176.2, 87.8)
- added LED22: LED, lib.pretty:INSW_LEDS, F.Cu at (195.3, 87.8)
- added LED23: LED, lib.pretty:INSW_LEDS, F.Cu at (214.3, 87.8)
- added LED24: LED, lib.pretty:INSW_LEDS, F.Cu at (233.4, 87.8)
- added LED25: LED, lib.pretty:INSW_LEDS, F.Cu at (252.4, 87.8)
- added LED26: LED, lib.pretty:INSW_LEDS, F.Cu at (271.5, 87.8)
- added LED27: LED, lib.pretty:INSW_LEDS, F.Cu at (290.5, 87.8)
- added LED28: LED, lib.pretty:INSW_LEDS, F.Cu at (309.6, 87.8)
- added LED29: LED, lib.pretty:INSW_LEDS, F.Cu at (333.4, 87.8)
- added LED3: LED, lib.pretty:INSW_LEDS, F.Cu at (109.5, 68.7)
- added LED30: LED, lib.pretty:INSW_LEDS, F.Cu at (78.6, 106.8)
- added LED31: LED, lib.pretty:INSW_LEDS, F.Cu at (104.8, 106.8)
- added LED32: LED, lib.pretty:INSW_LEDS, F.Cu at (123.8, 106.8)
- added LED33: LED, lib.pretty:INSW_LEDS, F.Cu at (142.9, 106.8)
- added LED34: LED, lib.pretty:INSW_LEDS, F.Cu at (161.9, 106.8)
- added LED35: LED, lib.pretty:INSW_LEDS, F.Cu at (181.0, 106.8)
- added LED36: LED, lib.pretty:INSW_LEDS, F.Cu at (200.0, 106.8)
- added LED37: LED, lib.pretty:INSW_LEDS, F.Cu at (219.1, 106.8)
- added LED38: LED, lib.pretty:INSW_LEDS, F.Cu at (238.1, 106.8)
- added LED39: LED, lib.pretty:INSW_LEDS, F.Cu at (257.2, 106.8)
- added LED4: LED, lib.pretty:INSW_LEDS, F.Cu at (128.6, 68.7)
- added LED40: LED, lib.pretty:INSW_LEDS, F.Cu at (276.2, 106.8)
- added LED41: LED, lib.pretty:INSW_LEDS, F.Cu at (295.3, 106.8)
- added LED42: LED, lib.pretty:INSW_LEDS, F.Cu at (326.2, 106.8)
- added LED43: LED, lib.pretty:INSW_LEDS, F.Cu at (83.3, 125.9)
- added LED44: LED, lib.pretty:INSW_LEDS, F.Cu at (114.3, 125.9)
- added LED45: LED, lib.pretty:INSW_LEDS, F.Cu at (133.3, 125.9)
- added LED46: LED, lib.pretty:INSW_LEDS, F.Cu at (152.4, 125.9)
- added LED47: LED, lib.pretty:INSW_LEDS, F.Cu at (171.4, 125.9)
- added LED48: LED, lib.pretty:INSW_LEDS, F.Cu at (190.5, 125.9)
- added LED49: LED, lib.pretty:INSW_LEDS, F.Cu at (209.6, 125.9)
- added LED5: LED, lib.pretty:INSW_LEDS, F.Cu at (147.6, 68.7)
- added LED50: LED, lib.pretty:INSW_LEDS, F.Cu at (228.6, 125.9)
- added LED51: LED, lib.pretty:INSW_LEDS, F.Cu at (247.7, 125.9)
- added LED52: LED, lib.pretty:INSW_LEDS, F.Cu at (266.7, 125.9)
- added LED53: LED, lib.pretty:INSW_LEDS, F.Cu at (285.8, 125.9)
- added LED54: LED, lib.pretty:INSW_LEDS, F.Cu at (311.9, 125.9)
- added LED55: LED, lib.pretty:INSW_LEDS, F.Cu at (338.1, 125.9)
- added LED56: LED, lib.pretty:INSW_LEDS, F.Cu at (73.8, 144.9)
- added LED57: LED, lib.pretty:INSW_LEDS, F.Cu at (97.6, 144.9)
- added LED58: LED, lib.pretty:INSW_LEDS, F.Cu at (121.4, 144.9)
- added LED59: LED, lib.pretty:INSW_LEDS, F.Cu at (192.9, 144.9)
- added LED6: LED, lib.pretty:INSW_LEDS, F.Cu at (166.7, 68.7)
- added LED60: LED, lib.pretty:INSW_LEDS, F.Cu at (264.3, 144.9)
- added LED61: LED, lib.pretty:INSW_LEDS, F.Cu at (288.1, 144.9)
- added LED62: LED, lib.pretty:INSW_LEDS, F.Cu at (309.6, 144.9)
- added LED63: LED, lib.pretty:INSW_LEDS, F.Cu at (333.4, 144.9)
- added LED64: LED, lib.pretty:LED-0603, B.Cu at (163.7, 144.3)
- added LED7: LED, lib.pretty:INSW_LEDS, F.Cu at (185.7, 68.7)
- added LED8: LED, lib.pretty:INSW_LEDS, F.Cu at (204.8, 68.7)
- added LED9: LED, lib.pretty:INSW_LEDS, F.Cu at (223.8, 68.7)
- added Q1: TC1264, lib.pretty:SOT-223, B.Cu at (100.0, 131.0)
- added R4: 4.7k, lib.pretty:SMD-1005, B.Cu at (217.3, 141.4)
- added R5: 20k, lib.pretty:SMD-1005, B.Cu at (218.9, 154.0)
- added R6: 4.7k, lib.pretty:SMD-1005, B.Cu at (220.0, 154.0)
- added R7: 100k, lib.pretty:SMD-1005, B.Cu at (221.1, 154.0)
- added R8: 1k, lib.pretty:SMD-1005, B.Cu at (166.3, 144.8)
- added S154: SW, lib.pretty:MXALPS_HIDDEN, F.Cu at (321.5, 131.0)
- added U2: IS31FL3731C, lib.pretty:SSOP-28, B.Cu at (218.0, 147.7)
- C1: value 2.2u -> 1uF
- C2: value 2.2u -> 0.22uF
- C3, C6: value 100n -> 0.1uF
- C4, C5: value 100n -> 1uF
- IC_LOGO: moved to B.Cu
- P2: value CONN_2 -> CONN_11; footprint lib.pretty:HEADER_1x2 -> lib.pretty:HEADER_1x11
- R3: value 1k -> 4.7k
- S64: value TAC_SWITCHSMD_EVQP2 -> TAC_SWITCH
- U1: value MK20LF -> MK20DX128VLF5
- moved R2 102.8 mm to (148.9, 149.4), turned to 270 degrees
- moved R1 102.8 mm to (148.9, 148.2), turned to 270 degrees
- moved R3 66.4 mm to (216.2, 141.4)
- moved C5 64.0 mm to (96.0, 131.0), turned to 0 degrees
- moved C1 62.6 mm to (103.9, 131.0)
- moved C4 58.2 mm to (222.3, 154.0), turned to 0 degrees
- moved C3 49.9 mm to (213.9, 141.4), turned to 0 degrees
- moved C2 49.2 mm to (215.0, 141.4)
- moved IC_LOGO 20.9 mm to (243.1, 144.2), turned to 180 degrees
- moved D60 17.3 mm to (257.2, 145.3), turned to 180 degrees
- moved D63 16.7 mm to (326.2, 150.0), turned to 180 degrees
- moved D62 16.7 mm to (302.4, 150.0), turned to 180 degrees
- moved D61 16.7 mm to (281.0, 150.0), turned to 180 degrees
- moved D58 16.7 mm to (114.3, 150.0), turned to 180 degrees
- moved D59 16.7 mm to (185.7, 150.0), turned to 180 degrees
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- renumbered P3 to P1, Ss15 to S114, Ss56 to S156, Ss57 to S157, Ss58 to S158, Ss59 to S159, Ss60 to S160, Ss61 to S161, Ss62 to S162, Ss63 to S163
Connections:
- net /matrix/Col9 renamed /mcu/PTD0
- net /mcu/GND renamed /mcu/SHLD
- C1 pad 1: VDD -> +5V
- C2 pad 1: +5V -> Net-(C2-Pad1)
- C2 pad 2: VSS -> /mcu/AUD
- C3 pad 1: VDD -> Net-(C3-Pad1)
- C4 pad 1: VDDA -> VSS
- C4 pad 2: VSSA -> VDD
- C6 pad 1: /mcu/RST -> VDD
- J1 pad 4: (no net) -> Net-(J1-Pad4)
- P1 pad 10: /mcu/RST -> /mcu/MCU_RESET
- P1 pad 7: /mcu/TX0 -> Net-(P1-Pad7)
- P1 pad 9: (no net) -> Net-(P1-Pad9)
- P2 pad 1: /mcu/RX0 -> VDD
- P2 pad 2: /mcu/TX0 -> /mcu/SWD_DIO
- R3 pad 1: Net-(D64-Pad2) -> VDD
- R3 pad 2: VSS -> /mcu/SDA0
- S1 pad 1: /matrix/Col1 -> /mcu/PTC0
- S10 pad 1: /matrix/Col1 -> /mcu/PTC0
- S11 pad 1: /matrix/Col2 -> /mcu/PTC1
- S114 pad 1: /matrix/Col6 -> /mcu/PTC4
- S114 pad 2: Net-(D15-Pad1) -> Net-(D14-Pad1)
- S12 pad 1: /matrix/Col3 -> /mcu/PTC2
- S13 pad 1: /matrix/Col4 -> /mcu/PTC3
- S14 pad 1: /matrix/Col5 -> /mcu/PTC4
- S15 pad 1: /matrix/Col6 -> /mcu/PTC5
- S156 pad 1: /matrix/Col2 -> /mcu/PTC1
- S157 pad 1: /matrix/Col3 -> /mcu/PTC2
- S158 pad 1: /matrix/Col4 -> /mcu/PTC3
- S159 pad 1: /matrix/Col5 -> /mcu/PTC4
- S16 pad 1: /matrix/Col7 -> /mcu/PTC6
- S160 pad 1: /matrix/Col6 -> /mcu/PTC5
- S161 pad 1: /matrix/Col7 -> /mcu/PTC6
- S162 pad 1: /matrix/Col8 -> /mcu/PTC7
- S17 pad 1: /matrix/Col8 -> /mcu/PTC7
- S19 pad 1: /matrix/Col1 -> /mcu/PTC0
- S2 pad 1: /matrix/Col2 -> /mcu/PTC1
- S20 pad 1: /matrix/Col2 -> /mcu/PTC1
- S21 pad 1: /matrix/Col3 -> /mcu/PTC2
- S22 pad 1: /matrix/Col4 -> /mcu/PTC3
- S23 pad 1: /matrix/Col5 -> /mcu/PTC4
- S24 pad 1: /matrix/Col6 -> /mcu/PTC5
- S25 pad 1: /matrix/Col7 -> /mcu/PTC6
- S26 pad 1: /matrix/Col8 -> /mcu/PTC7
- S28 pad 1: /matrix/Col1 -> /mcu/PTC0
- S29 pad 1: /matrix/Col2 -> /mcu/PTC1
- S3 pad 1: /matrix/Col3 -> /mcu/PTC2
- S30 pad 1: /matrix/Col3 -> /mcu/PTC2
- S31 pad 1: /matrix/Col4 -> /mcu/PTC3
- S32 pad 1: /matrix/Col5 -> /mcu/PTC4
- S33 pad 1: /matrix/Col6 -> /mcu/PTC5
- S34 pad 1: /matrix/Col7 -> /mcu/PTC6
- S35 pad 1: /matrix/Col8 -> /mcu/PTC7
- S37 pad 1: /matrix/Col1 -> /mcu/PTC0
- S38 pad 1: /matrix/Col2 -> /mcu/PTC1
- S39 pad 1: /matrix/Col3 -> /mcu/PTC2
- S4 pad 1: /matrix/Col4 -> /mcu/PTC3
- S40 pad 1: /matrix/Col4 -> /mcu/PTC3
- S41 pad 1: /matrix/Col5 -> /mcu/PTC4
- S42 pad 1: /matrix/Col6 -> /mcu/PTC5
- S43 pad 1: /matrix/Col7 -> /mcu/PTC6
- S44 pad 1: /matrix/Col8 -> /mcu/PTC7
- S46 pad 1: /matrix/Col1 -> /mcu/PTC0
- S47 pad 1: /matrix/Col2 -> /mcu/PTC1
- S48 pad 1: /matrix/Col3 -> /mcu/PTC2
- S49 pad 1: /matrix/Col4 -> /mcu/PTC3
- S5 pad 1: /matrix/Col5 -> /mcu/PTC4
- S50 pad 1: /matrix/Col5 -> /mcu/PTC4
- S51 pad 1: /matrix/Col6 -> /mcu/PTC5
- S52 pad 1: /matrix/Col7 -> /mcu/PTC6
- S53 pad 1: /matrix/Col8 -> /mcu/PTC7
- S55 pad 1: /matrix/Col1 -> /mcu/PTC0
- S56 pad 1: /matrix/Col2 -> /mcu/PTC1
- S57 pad 1: /matrix/Col3 -> /mcu/PTC2
- S58 pad 1: /matrix/Col4 -> /mcu/PTC3
- S59 pad 1: /matrix/Col5 -> /mcu/PTC4
- S6 pad 1: /matrix/Col6 -> /mcu/PTC5
- S60 pad 1: /matrix/Col6 -> /mcu/PTC5
- S61 pad 1: /matrix/Col7 -> /mcu/PTC6
- S62 pad 1: /matrix/Col8 -> /mcu/PTC7
- S64 pad 1: /mcu/RST -> Net-(S64-Pad1)
- S64 pad 2: VSS -> /mcu/MCU_RESET
- S64 pad 3: (no net) -> VSS
- S7 pad 1: /matrix/Col7 -> /mcu/PTC6
- S8 pad 1: /matrix/Col8 -> /mcu/PTC7
- U1 pad 10: VDDA -> Net-(U1-Pad10)
- U1 pad 11: VSSA -> Net-(U1-Pad11)
- U1 pad 12: VSSA -> Net-(U1-Pad12)
- U1 pad 13: (no net) -> Net-(U1-Pad13)
- U1 pad 14: (no net) -> Net-(U1-Pad14)
- U1 pad 15: (no net) -> Net-(U1-Pad15)
- U1 pad 21: (no net) -> /mcu/PTA4
- U1 pad 24: (no net) -> /mcu/PTA18
- U1 pad 26: /mcu/RST -> /mcu/MCU_RESET
- U1 pad 27: /matrix/Col1 -> /mcu/SCL0
- U1 pad 28: /matrix/Col2 -> /mcu/SDA0
- U1 pad 29: /matrix/Col3 -> /mcu/PTB2
- U1 pad 30: /matrix/Col4 -> /mcu/PTB3
- U1 pad 31: /matrix/Col5 -> /mcu/SDB
- U1 pad 32: /matrix/Col6 -> /mcu/INTB
- U1 pad 33: (no net) -> /mcu/PTC0
- U1 pad 34: (no net) -> /mcu/PTC1
- U1 pad 35: (no net) -> /mcu/PTC2
- U1 pad 36: (no net) -> /mcu/PTC3
- U1 pad 37: /matrix/Col7 -> /mcu/PTC4
- U1 pad 38: /matrix/Col8 -> /mcu/PTC5
- U1 pad 39: (no net) -> /mcu/PTC6
- U1 pad 40: (no net) -> /mcu/PTC7
- U1 pad 6: +5V -> VDD
- U1 pad 7: (no net) -> /mcu/ADC0_DP0
- U1 pad 8: (no net) -> /mcu/ADC0_DM0
- U1 pad 9: VDDA -> Net-(U1-Pad9)
Routing:
- net /ledmatrix/CA2: track 0.00 -> 622.1 mm, vias 0 -> 2
- net /ledmatrix/CA8: track 0.00 -> 588.3 mm
- net /ledmatrix/CA4: track 0.00 -> 550.2 mm
- net /ledmatrix/CA7: track 0.00 -> 545.5 mm, vias 0 -> 4
- net /ledmatrix/CA1: track 0.00 -> 544.5 mm
- net /mcu/PTC1: track 0.00 -> 518.3 mm, vias 0 -> 2
- net /ledmatrix/CA6: track 0.00 -> 508.6 mm, vias 0 -> 2
- net /ledmatrix/CA3: track 0.00 -> 490.6 mm, vias 0 -> 1
- net /ledmatrix/CA9: track 0.00 -> 484.6 mm, vias 0 -> 2
- net /ledmatrix/CA5: track 0.00 -> 449.4 mm
- net /mcu/PTC6: track 0.00 -> 446.1 mm, vias 0 -> 1
- net /mcu/PTC0: track 0.00 -> 441.0 mm, vias 0 -> 2
- net /matrix/Col2: track 440.1 -> 0.00 mm, vias 2 -> 0
- net /matrix/Col6: track 428.5 -> 0.00 mm
- net /mcu/PTC3: track 0.00 -> 424.7 mm, vias 0 -> 3
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Other:
- board text added: "AUD"
- board text added: "IC60 1.1a"
- board text added: "RST"
- board text added: "SCL0"
- board text added: "SDA0"
- board text added: "VDD"
- board text removed: "IC60 1.03a"
