File: WhiteFox/WhiteFox.kicad_pcb (KiCad board)
At the start: 2 copper layers, 304.8 x 95.3 mm, 291 parts, among them J1 USB_CONN, P1 FLASH_HDR, P2 CONN_11, Q1 TC1264, U1 MK20DX256VLH7, U2 IS31FL3731C, X1 CRYSTAL

Commit message: WhiteFox 1.1c
Parts:
- added C10: 0.1uF, footprints:SMD-0402, B.Cu at (212.2, 169.3)
- added D72: ESD_BIDIR_1CH, footprints:SMD-0402, B.Cu at (68.3, 82.4)
- added D73: ESD_BIDIR_1CH, footprints:SMD-0402, B.Cu at (71.5, 82.4)
- added H1: 1PIN, footprints:1PAD_5.5, F.Cu at (80.6, 123.8)
- added R11: 5.1k, footprints:SMD-0402, B.Cu at (72.4, 81.0)
- added R12: 5.1k, footprints:SMD-0402, B.Cu at (67.6, 81.0)
- added U2: MK20DX256VMC7R, footprints:MAPBGA121, B.Cu at (216.0, 160.4)
- C1, C2, C3, C4, C5, C6, C7, C8, C9, R1, R10, R2, R3, R4, R5, R6, R7, R8, R9: footprint lib.pretty:SMD-1005 -> footprints:SMD-0402
- D1, D10, D11, D12, D13, D14, D15, D16, D17, D18, D19, D2, D20, D21, D22, D23, D24, D25, D26, D27, D28, D29, D3, D30, D31, D32, D33, D34, D35, D36, D37, D38, D39, D4, D40, D41, D42, D43, D44, D45, D46, D47, D48, D49, D5, D50, D51, D52, D53, D54, D55, D56, D57, D58, D59, D6, D60, D61, D62, D63, D64, D65, D66, D67, D68, D69, D7, D70, D71, D8, D9: footprint lib.pretty:SOT123-DIODE -> footprints:SOT123-DIODE
- FID1, FID2, FID3: footprint lib.pretty:FID -> footprints:FID
- G***: footprint lib.pretty:FOXY_LOGO -> footprints:FOXY_LOGO
- IC_LOGO: footprint lib.pretty:IC_LOGO -> footprints:IC_LOGO
- J1: value USB_CONN -> USBC; footprint lib.pretty:USB2_MICROB_WURTH -> footprints:E8124-010-01
- LED1, LED10, LED11, LED12, LED13, LED14, LED15, LED16, LED17, LED18, LED19, LED2, LED20, LED21, LED22, LED23, LED24, LED25, LED26, LED27, LED28, LED29, LED3, LED30, LED31, LED32, LED33, LED34, LED35, LED36, LED37, LED38, LED39, LED4, LED40, LED41, LED42, LED43, LED44, LED45, LED46, LED47, LED48, LED49, LED5, LED50, LED51, LED52, LED53, LED54, LED55, LED56, LED57, LED58, LED59, LED6, LED60, LED61, LED62, LED63, LED64, LED65, LED66, LED67, LED68, LED69, LED7, LED70, LED71, LED8, LED9: footprint lib.pretty:INSW_LEDS -> footprints:INSW_LEDS
- LED115, LED145, LED147, LED159, LED162, LED163, LED164, LED165, LED166, LED167, LED168, LED245, LED263, LED265, LED266: footprint lib.pretty:INSW_LEDS_HIDDEN -> footprints:INSW_LEDS_HIDDEN
- LED72: footprint lib.pretty:LED-0603 -> footprints:LED-0603
- P1: footprint lib.pretty:JLINK_NEEDLE -> footprints:JLINK_NEEDLE
- P2: footprint lib.pretty:HEADER_1x11 -> footprints:HEADER_1x11
- Q1: footprint lib.pretty:SOT-223 -> footprints:SOT-223
- S1, S10, S11, S12, S13, S14, S15, S16, S17, S18, S19, S2, S20, S21, S22, S23, S24, S25, S26, S27, S28, S29, S3, S30, S31, S32, S33, S34, S35, S36, S37, S38, S39, S4, S40, S41, S42, S43, S44, S45, S46, S47, S48, S49, S5, S50, S51, S52, S53, S54, S55, S56, S57, S58, S59, S6, S60, S61, S62, S63, S64, S65, S66, S67, S68, S69, S7, S70, S71, S8, S9: footprint lib.pretty:MX -> footprints:MX
- S115, S145, S147, S159, S162, S163, S164, S165, S166, S167, S168, S245, S263, S265, S266: footprint lib.pretty:MX_HIDDEN -> footprints:MX_HIDDEN
- S72: footprint lib.pretty:TACT_5.2x5.2 -> footprints:TACT_5.2x5.2
- STAB1, STAB10, STAB11, STAB12, STAB13, STAB14, STAB15, STAB2, STAB3, STAB4, STAB5, STAB6, STAB7, STAB8, STAB9: footprint lib.pretty:STAB -> footprints:STAB
- U1: footprint lib.pretty:LQFP64 -> footprints:LQFP64
- U3: renamed from U2; footprint lib.pretty:SSOP-28 -> footprints:SSOP-28
- X1: footprint lib.pretty:NX3225SA -> footprints:NX3225SA
- moved C1 12.2 mm to (75.2, 111.3), turned to 90 degrees
- moved C2 9.72 mm to (75.2, 119.6), turned to 90 degrees
- moved Q1 9.36 mm to (75.2, 115.5), turned to 270 degrees
- moved C5 0.54 mm to (219.2, 168.5), turned to 180 degrees
- moved J1 0.20 mm to (69.8, 76.4)
- turned R4 to 270 degrees
Connections:
- net /mcu/PTB18 renamed /Col3
- net /mcu/PTB19 renamed /Col4
- net /mcu/PTB2 renamed /Col1
- net /mcu/PTB3 renamed /Col2
- net /mcu/PTC0 renamed /Col5
- net /mcu/PTC1 renamed /Row7
- net /mcu/PTC10 renamed /Col8
- net /mcu/PTC11 renamed /Col9
- net /mcu/PTC2 renamed /Row8
- net /mcu/PTC8 renamed /Col6
- net /mcu/PTC9 renamed /Col7
- net /mcu/PTD0 renamed /Row1
- net /mcu/PTD1 renamed /Row2
- net /mcu/PTD4 renamed /Row3
- net /mcu/PTD5 renamed /Row4
- net /mcu/PTD6 renamed /Row5
- net /mcu/PTD7 renamed /Row6
- net Net-(R3-Pad1) renamed /mcu/PTA0
- net Net-(R4-Pad1) renamed /mcu/PTA3
- net Net-(U1-Pad32) renamed /mcu/EXTAL0
- net Net-(U1-Pad33) renamed /mcu/XTAL0
- J1 pad 1: +5V -> VSS
- J1 pad 4: (no net) -> +5V
- J1 pad 5: VSS -> Net-(J1-Pad5)
- R1 pad 1: Net-(J1-Pad2) -> /mcu/USB_DM
- R1 pad 2: /mcu/USB_DM -> /mcu/USB0_DM
- R2 pad 1: Net-(J1-Pad3) -> /mcu/USB_DP
- R2 pad 2: /mcu/USB_DP -> /mcu/USB0_DP
- S72 pad 1: (no net) -> Net-(S72-Pad1)
- U1 pad 1: (no net) -> Net-(U1-Pad1)
- U1 pad 10: (no net) -> Net-(U1-Pad10)
- U1 pad 11: (no net) -> Net-(U1-Pad11)
- U1 pad 12: (no net) -> Net-(U1-Pad12)
- U1 pad 13: (no net) -> Net-(U1-Pad13)
- U1 pad 14: (no net) -> Net-(U1-Pad14)
- U1 pad 15: (no net) -> Net-(U1-Pad15)
- U1 pad 16: (no net) -> Net-(U1-Pad16)
- U1 pad 17: (no net) -> Net-(U1-Pad17)
- U1 pad 18: (no net) -> Net-(U1-Pad18)
- U1 pad 19: (no net) -> Net-(U1-Pad19)
- U1 pad 2: (no net) -> Net-(U1-Pad2)
- U1 pad 20: (no net) -> Net-(U1-Pad20)
- U1 pad 26: (no net) -> Net-(U1-Pad26)
- U1 pad 28: (no net) -> Net-(U1-Pad28)
- U1 pad 29: (no net) -> Net-(U1-Pad29)
- U1 pad 46: (no net) -> Net-(U1-Pad46)
- U1 pad 49: (no net) -> Net-(U1-Pad49)
- U1 pad 5: /mcu/USB_DP -> /mcu/USB0_DP
- U1 pad 50: (no net) -> Net-(U1-Pad50)
- U1 pad 51: (no net) -> Net-(U1-Pad51)
- U1 pad 52: (no net) -> Net-(U1-Pad52)
- U1 pad 6: /mcu/USB_DM -> /mcu/USB0_DM
- U1 pad 9: (no net) -> Net-(U1-Pad9)
- U3 pad 10: (no net) -> /mcu/CB4
- U3 pad 11: (no net) -> /mcu/CB5
- U3 pad 12: (no net) -> /mcu/CB6
- U3 pad 13: (no net) -> /mcu/CB7
- U3 pad 14: (no net) -> /mcu/CB8
- U3 pad 15: (no net) -> /mcu/CB9
- U3 pad 7: (no net) -> /mcu/CB1
- U3 pad 8: (no net) -> /mcu/CB2
- U3 pad 9: (no net) -> /mcu/CB3
Routing:
- net Net-(J1-Pad3): track 172.3 -> 0.00 mm, vias 2 -> 0
- net Net-(J1-Pad2): track 171.8 -> 0.00 mm, vias 2 -> 0
- net /mcu/USB_DP: track 2.07 -> 170.9 mm
- net /mcu/USB_DM: track 2.58 -> 170.0 mm, vias 0 -> 1
- net /Col6: track 534.8 -> 450.9 mm, vias 2 -> 7
- net /Col5: track 544.8 -> 470.0 mm, vias 1 -> 6
- net /Col1: track 528.9 -> 459.5 mm, vias 1 -> 5
- net /ledmatrix/CA8: track 554.5 -> 488.1 mm, vias 0 -> 4
- net /ledmatrix/CA4: track 556.1 -> 491.2 mm, vias 2 -> 7
- net /Col2: track 534.8 -> 473.2 mm, vias 2 -> 6
- net /ledmatrix/CA5: track 501.8 -> 441.6 mm, vias 3 -> 5
- net /ledmatrix/CA6: track 546.3 -> 489.7 mm, vias 2 -> 5
- net /Col9: track 465.6 -> 425.2 mm, vias 1 -> 7
- net /ledmatrix/CA2: track 524.0 -> 483.7 mm, vias 2 -> 5
- net /Col7: track 480.2 -> 441.9 mm, vias 2 -> 5
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- added copper zone on B.Cu, net /mcu/SHLD
- added copper zone on F.Cu, net /mcu/SHLD
Other:
- board size 304.8 x 95.3 mm -> 304.8 x 101.1 mm
- net class 4mil added: clearance 0.1016, trace_width 0.1016, via_dia 0.3556, via_drill 0.2032
- net class Default: clearance 0.1524 -> 0.1016; trace_width 0.1524 -> 0.25; via_dia 0.6096 -> 0.3556; via_drill 0.508 -> 0.2032
- net class GND removed
- net class Power: clearance 0.1524 -> 0.1016; via_dia 0.6096 -> 0.508; via_drill 0.508 -> 0.3048
- net class Shield added: clearance 0.1016, trace_width 0.508, via_dia 0.508, via_drill 0.3048
- rule trace_clearance: 0.1524 -> 0.1016
- rule trace_min: 0.0254 -> 0.1016
- rule via_min_size: 0.4064 -> 0.3556
- board text added: "WF 1.1c"
- board text removed: "WF 1.02a"
